File: rj45-trs.kicad_sch (KiCad schematic)
At the start: 5 parts, among them J101 NSJ12HC, J102 NSJ12HC, J103 NE8FAH

Commit message: Refresh
Parts:
- ICON101: footprint V2_Artwork:Logo_Tiny -> V2_Artwork:Logo_Small
- J101, J102: Mouser (none) -> 568-NSJ12HC
- J103: Mouser (none) -> 568-NE8FAH
Changed lines of the file:
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@@
+			)
+		)
+		(property "Mouser" "568-NSJ12HC"
+			(at 179.07 152.146 0)
+			(effects
+				(font
+					(size 1.27 1.27)
+				)
+				(hide yes)
 			)
 		)
@@
 			)
 		)
+		(property "Mouser" "568-NSJ12HC"
+			(at 179.07 120.396 0)
+			(effects
+				(font
+					(size 1.27 1.27)
+				)
+				(hide yes)
+			)
+		)
 		(pin "G"
 		)
@@
 			)
 		)
+		(property "Mouser" "568-NSJ12HC"
+			(at 220.98 120.396 0)
+			(effects
+				(font
+					(size 1.27 1.27)
+				)
+				(hide yes)
+			)
+		)
 		(pin "T2"
 		)
@@
 		(at 266.7 176.53 0)
 		(unit 1)
-		(exclude_from_sim yes)
+		(exclude_from_sim no)
 		(in_bom no)
 		(on_board yes)
@@
 		)
 		(property "Description" ""
+			(at 266.7 176.53 0)
+			(effects
+				(font
+					(size 1.27 1.27)
+				)
+				(hide yes)
+			)
+		)
+		(property "Sim.Enable" "0"
 			(at 266.7 176.53 0)
 			(effects
@@
 		(at 71.12 105.41 0)
 		(unit 1)
-		(exclude_from_sim yes)
+		(exclude_from_sim no)
 		(in_bom yes)
 		(on_board yes)
@@
 		(property "Description" ""
 			(at 71.12 105.41 0)
+			(effects
+				(font
+					(size 1.27 1.27)
+				)
+				(hide yes)
+			)
+		)
+		(property "Mouser" "568-NE8FAH"
+			(at 71.12 132.842 0)
 			(effects
 				(font
@@
 			)
 		)
+		(property "Mouser" "568-NSJ12HC"
+			(at 220.98 152.146 0)
+			(effects
+				(font
+					(size 1.27 1.27)
+				)
+				(hide yes)
+			)
+		)
 		(pin "T2"
 		)
@@
 		(at 241.3 176.53 0)
 		(unit 1)
-		(exclude_from_sim yes)
+		(exclude_from_sim no)
 		(in_bom no)
 		(on_board yes)
@@
 			)
 		)
-		(property "Footprint" "V2_Artwork:Logo_Tiny"
+		(property "Footprint" "V2_Artwork:Logo_Small"
 			(at 241.3 184.15 0)
 			(effects
@@
 			(at 241.3 176.53 0)
 			(effects
+				(font
+					(size 1.27 1.27)
+				)
+				(hide yes)
+			)
+		)
+		(property "Sim.Enable" "0"
+			(at 241.3 176.53 0)
+			(effects

Commit message: Update parts
Parts:
- J101, J102: Manufacturer (none) -> Neutrik; Product (none) -> NSJ12HC
- J103: Manufacturer (none) -> Neutrik; Product (none) -> NE8FAH
Changed lines of the file:
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@@
 	)
 	(symbol
-		(lib_id "power:GND")
+		(lib_id "V2_power:GND")
 		(at 215.9 116.84 270)
 		(mirror x)
@@
 			)
 		)
+		(property "Manufacturer" "Neutrik"
+			(at 179.07 154.94 0)
+			(effects
+				(font
+					(size 1.27 1.27)
+				)
+				(hide yes)
+			)
+		)
+		(property "Product" "NSJ12HC"
+			(at 179.07 152.4 0)
+			(effects
+				(font
+					(size 1.27 1.27)
+				)
+				(hide yes)
+			)
+		)
 		(pin "G"
 		)
@@
 	)
 	(symbol
-		(lib_id "power:GND")
+		(lib_id "V2_power:GND")
 		(at 77.47 74.93 90)
 		(unit 1)
@@
 	)
 	(symbol
-		(lib_id "power:GND")
+		(lib_id "V2_power:GND")
 		(at 220.98 102.87 0)
 		(mirror y)
@@
 			)
 		)
+		(property "Manufacturer" "Neutrik"
+			(at 179.07 123.19 0)
+			(effects
+				(font
+					(size 1.27 1.27)
+				)
+				(hide yes)
+			)
+		)
+		(property "Product" "NSJ12HC"
+			(at 179.07 120.65 0)
+			(effects
+				(font
+					(size 1.27 1.27)
+				)
+				(hide yes)
+			)
+		)
 		(pin "G"
 		)
@@
 			)
 		)
+		(property "Manufacturer" "Neutrik"
+			(at 220.98 123.19 0)
+			(effects
+				(font
+					(size 1.27 1.27)
+				)
+				(hide yes)
+			)
+		)
+		(property "Product" "NSJ12HC"
+			(at 220.98 120.65 0)
+			(effects
+				(font
+					(size 1.27 1.27)
+				)
+				(hide yes)
+			)
+		)
 		(pin "T2"
 		)
@@
 			)
 		)
-		(property "Sim.Enable" "0"
-			(at 266.7 176.53 0)
-			(effects
-				(font
-					(size 1.27 1.27)
-				)
-				(hide yes)
-			)
-		)
 		(instances
 			(project "express"
@@
 	)
 	(symbol
-		(lib_id "power:GND")
+		(lib_id "V2_power:GND")
 		(at 179.07 102.87 0)
 		(mirror y)
@@
 	)
 	(symbol
-		(lib_id "power:GND")
+		(lib_id "V2_power:GND")
 		(at 71.12 118.11 0)
 		(mirror y)
@@
 	)
 	(symbol
-		(lib_id "power:GND")
+		(lib_id "V2_power:GND")
 		(at 215.9 85.09 270)
 		(mirror x)
@@
 		(property "Mouser" "568-NE8FAH"
 			(at 71.12 132.842 0)
+			(effects
+				(font
+					(size 1.27 1.27)
+				)
+				(hide yes)
+			)
+		)
+		(property "Manufacturer" "Neutrik"
+			(at 71.12 133.35 0)
+			(effects
+				(font
+					(size 1.27 1.27)
+				)
+				(hide yes)
+			)
+		)
+		(property "Product" "NE8FAH"
+			(at 71.12 135.89 0)
 			(effects
 				(font
@@
 			)
 		)
+		(property "Manufacturer" "Neutrik"
+			(at 220.98 154.94 0)
+			(effects
+				(font
+					(size 1.27 1.27)
+				)
+				(hide yes)
+			)
+		)
+		(property "Product" "NSJ12HC"
+			(at 220.98 152.4 0)
+			(effects
+				(font
+					(size 1.27 1.27)
+				)
+				(hide yes)
+			)
+		)
 		(pin "T2"
 		)
@@
 	)
 	(symbol
-		(lib_id "power:GND")
+		(lib_id "V2_power:GND")
 		(at 173.99 85.09 270)
 		(mirror x)
@@
 	)
 	(symbol
-		(lib_id "power:PWR_FLAG")
+		(lib_id "V2_power:PWR_FLAG")
 		(at 77.47 74.93 90)
 		(unit 1)
@@
 	)
 	(symbol
-		(lib_id "power:GND")
+		(lib_id "V2_power:GND")
 		(at 173.99 116.84 270)
 		(mirror x)
@@
 				)
 				(justify left)
-			)
-		)
+				(hide yes)
+			)
+		)
